Commit message: inizializzata platform, ancora non sono in grado di visualizzarla graficamente su rviz

File: urdf/mivia_rover.materials.xacro (robot description, xacro)
@@ -10,8 +10,8 @@
   </material>
   <!-- Optional greys for minor components (future-proofing) -->
-  <material name="mivia_dark_grey">
+  <material name="mivia_dark_gray">
     <color rgba="0.08 0.08 0.08 1.0"/>
   </material>
-  <material name="mivia_grey">
+  <material name="mivia_gray">
     <color rgba="0.25 0.25 0.25 1.0"/>
   </material>

File: urdf/mivia_rover_description.urdf.xacro (robot description, xacro)
@@ -5,4 +5,5 @@
     PLACEHOLDER: adapt naming conventions, frames, and ROS 2 control integration as needed.
   -->
+  <xacro:include filename="$(find mivia_rover_description)/urdf/mivia_rover.materials.xacro"/>
   <xacro:macro name="mivia_rover" params="prefix">
     <!-- ========================= -->
