Commit message: adjusted informations

File: urdf/mivia_rover_description.urdf.xacro (robot description, xacro)
@@ -27,7 +27,7 @@
     <!-- Wheel placement relative to base_link -->
     <!-- Convention: x forward, y left, z up -->
-    <!-- PLACEHOLDER: set wheelbase/track to match your real chassis -->
-    <xacro:property name="wheelbase" value="0.26"/>  <!-- front-to-rear distance -->
-    <xacro:property name="track"     value="0.22"/>  <!-- left-to-right distance -->
+    <!-- DONE: set wheelbase/track to match your real chassis -->
+    <xacro:property name="wheelbase" value="0.216"/>  <!-- front-to-rear distance -->
+    <xacro:property name="track"     value="0.355"/>  <!-- left-to-right distance -->
     <!-- Vertical placement: wheel centers below base_link -->
     <!-- PLACEHOLDER: adjust based on where you want base_link (COM vs geometric center) -->
@@ -58,5 +58,5 @@
         </geometry>
         <!-- PLACEHOLDER: material/color -->
-        <material name="gray"/>
+        <material name="mivia_gray"/>
       </visual>
       <inertial>
@@ -92,5 +92,5 @@
             <cylinder length="${wheel_width}" radius="${wheel_radius}"/>
           </geometry>
-          <material name="black"/>
+          <material name="mivia_black"/>
         </visual>
         <inertial>

Commit message: adesso il rover può essere visualizzato correttamente, va solo fine-tunata la posizione della base

File: urdf/mivia_rover_description.urdf.xacro (robot description, xacro)
@@ -12,58 +12,60 @@
     <xacro:property name="PI" value="3.1415926535897931"/>
     <!-- Base geometry -->
-    <!-- DONE: set real chassis dimensions (meters) -->
     <xacro:property name="base_length" value="0.32"/>
     <xacro:property name="base_width"  value="0.24"/>
     <xacro:property name="base_height" value="0.10"/>
     <!-- Base mass/inertia -->
-    <!-- PLACEHOLDER: set real mass (kg) and verify inertia with CAD/mesh -->
     <xacro:property name="base_mass" value="8.0"/>
     <!-- Wheel geometry -->
-    <!-- DONE: set real wheel radius/width (meters) -->
     <xacro:property name="wheel_radius" value="0.085"/>
     <xacro:property name="wheel_width"  value="0.08"/>
     <!-- Wheel mass/inertia -->
-    <!-- PLACEHOLDER: set real wheel mass (kg) -->
     <xacro:property name="wheel_mass" value="0.8"/>
-    <!-- Wheel placement relative to base_link -->
-    <!-- Convention: x forward, y left, z up -->
-    <!-- DONE: set wheelbase/track to match your real chassis -->
-    <xacro:property name="wheelbase" value="0.216"/>  <!-- front-to-rear distance -->
-    <xacro:property name="track"     value="0.355"/>  <!-- left-to-right distance -->
-    <!-- Vertical placement: wheel centers below base_link -->
-    <!-- PLACEHOLDER: adjust based on where you want base_link (COM vs geometric center) -->
-    <xacro:property name="wheel_z" value="${-(base_height/2.0) + wheel_radius}"/>
+    <!-- Wheel placement -->
+    <xacro:property name="wheelbase" value="0.216"/>
+    <xacro:property name="track"     value="0.355"/>
+    <!-- Ground clearance between wheel contact point and chassis bottom -->
+    <xacro:property name="ground_clearance" value="0.0"/>
+    <!-- base_link is aligned with wheel hubs (axle plane).
+         Wheel centers are placed at z=0 in base_link frame. -->
+    <xacro:property name="wheel_z" value="0.0"/>
     <!-- Joint dynamics -->
-    <!-- PLACEHOLDER: tune damping/friction for sim stability vs realism -->
     <xacro:property name="wheel_joint_damping" value="0.2"/>
     <xacro:property name="wheel_joint_friction" value="0.0"/>
     <!-- Joint limits -->
-    <!-- PLACEHOLDER: set realistic effort/velocity for motors (SI units) -->
     <xacro:property name="wheel_joint_effort" value="20.0"/>
     <xacro:property name="wheel_joint_velocity" value="20.0"/>
     <!-- ========================= -->
-    <!-- Base Link                 -->
+    <!-- Base Footprint (root)     -->
+    <!-- ========================= -->
+    <link name="${prefix}base_footprint"/>
+    <!-- base_link is at wheel hub height above ground -->
+    <joint name="${prefix}base_footprint_joint" type="fixed">
+      <parent link="${prefix}base_footprint"/>
+      <child  link="${prefix}base_link"/>
+      <origin xyz="0 0 ${wheel_radius + ground_clearance}" rpy="0 0 0"/>
+    </joint>
+    <!-- ========================= -->
+    <!-- Base Link (chassis)       -->
     <!-- ========================= -->
     <link name="${prefix}base_link">
       <collision>
-        <origin xyz="0 0 0" rpy="0 0 0"/>
+        <!-- Shift chassis geometry upwards so base_link stays on wheel hub plane -->
+        <origin xyz="0 0 ${base_height/2.0}" rpy="0 0 0"/>
         <geometry>
-          <!-- PLACEHOLDER: optionally replace with mesh -->
           <box size="${base_length} ${base_width} ${base_height}"/>
         </geometry>
       </collision>
       <visual>
-        <origin xyz="0 0 0" rpy="0 0 0"/>
+        <origin xyz="0 0 ${base_height/2.0}" rpy="0 0 0"/>
         <geometry>
           <box size="${base_length} ${base_width} ${base_height}"/>
         </geometry>
-        <!-- PLACEHOLDER: material/color -->
         <material name="mivia_gray"/>
       </visual>
       <inertial>
-        <!-- PLACEHOLDER: set COM offset if base_link is not COM -->
-        <origin xyz="0 0 0" rpy="0 0 0"/>
+        <!-- Inertial origin aligned with chassis center (same shift as geometry) -->
+        <origin xyz="0 0 ${base_height/2.0}" rpy="0 0 0"/>
         <mass value="${base_mass}"/>
-        <!-- Box inertia around center -->
         <inertia
           ixx="${base_mass/12.0 * (base_width*base_width + base_height*base_height)}"
@@ -81,6 +83,4 @@
       <link name="${wheel_link_name}">
         <collision>
-          <!-- Cylinder axis is along +Z by default in URDF, rotate to align with wheel axle -->
-          <!-- PLACEHOLDER: verify axis convention with your simulator/control stack -->
           <origin xyz="0 0 0" rpy="${PI/2} 0 0"/>
           <geometry>
@@ -98,6 +98,4 @@
           <origin xyz="0 0 0" rpy="${PI/2} 0 0"/>
           <mass value="${wheel_mass}"/>
-          <!-- Solid cylinder inertia (about its center) -->
-          <!-- Axis convention: after rotation, izz corresponds to axle; validate for your use -->
           <inertia
             ixx="${wheel_mass/12.0 * (3.0*wheel_radius*wheel_radius + wheel_width*wheel_width)}"
@@ -113,8 +111,4 @@
     <!-- 4 Wheels: Links           -->
     <!-- ========================= -->
-    <!-- Naming convention:
-         fl = front-left, fr = front-right, rl = rear-left, rr = rear-right
-         PLACEHOLDER: rename if your code expects different joint names.
-    -->
     <xacro:mivia_wheel wheel_link_name="${prefix}wheel_fl"/>
     <xacro:mivia_wheel wheel_link_name="${prefix}wheel_fr"/>
@@ -124,9 +118,4 @@
     <!-- 4 Wheel Joints            -->
     <!-- ========================= -->
-    <!-- Wheel positions -->
-    <!-- Front axle at +wheelbase/2, Rear axle at -wheelbase/2
-         Left at +track/2, Right at -track/2
-         PLACEHOLDER: if your coordinate frame uses opposite y convention, swap signs.
-    -->
     <!-- Front-Left -->
     <joint name="${prefix}wheel_fl_joint" type="continuous">
@@ -134,5 +123,4 @@
       <child  link="${prefix}wheel_fl"/>
       <origin xyz="${ wheelbase/2.0} ${ track/2.0} ${wheel_z}" rpy="0 0 0"/>
-      <!-- PLACEHOLDER: axle direction (commonly y for wheels if wheel rolls around y) -->
       <axis xyz="0 1 0"/>
       <dynamics damping="${wheel_joint_damping}" friction="${wheel_joint_friction}"/>
@@ -166,20 +154,4 @@
       <limit effort="${wheel_joint_effort}" velocity="${wheel_joint_velocity}"/>
     </joint>
-    <!-- ========================= -->
-    <!-- Optional: base footprint  -->
-    <!-- ========================= -->
-    <!-- PLACEHOLDER: if using Nav2, you often want base_footprint on the ground projection -->
-    <!--
-    <link name="${prefix}base_footprint"/>
-    <joint name="${prefix}base_footprint_joint" type="fixed">
-      <parent link="${prefix}base_footprint"/>
-      <child link="${prefix}base_link"/>
-      <origin xyz="0 0 ${base_height/2.0}" rpy="0 0 0"/>
-    </joint>
-    -->
-    <!-- ========================= -->
-    <!-- Optional: sensors frames   -->
-    <!-- ========================= -->
-    <!-- PLACEHOLDER: add imu_link, lidar_link, camera_link, etc. with fixed joints -->
   </xacro:macro>
 </robot>

Commit message: Rover Platform adjusted

File: urdf/mivia_rover_description.urdf.xacro (robot description, xacro)
@@ -1,13 +1,6 @@
 <?xml version="1.0"?>
 <robot xmlns:xacro="http://www.ros.org/wiki/xacro">
-  <!--
-    mivia_rover: 4-wheel differential rover (4 independently driven wheels)
-    PLACEHOLDER: adapt naming conventions, frames, and ROS 2 control integration as needed.
-  -->
   <xacro:include filename="$(find mivia_rover_description)/urdf/mivia_rover.materials.xacro"/>
   <xacro:macro name="mivia_rover" params="prefix">
-    <!-- ========================= -->
-    <!-- Constants / Parameters    -->
-    <!-- ========================= -->
     <xacro:property name="PI" value="3.1415926535897931"/>
     <!-- Base geometry -->
@@ -25,8 +18,9 @@
     <xacro:property name="wheelbase" value="0.216"/>
     <xacro:property name="track"     value="0.355"/>
-    <!-- Ground clearance between wheel contact point and chassis bottom -->
+    <!-- Optional clearance of wheel contact point w.r.t. base_footprint -->
     <xacro:property name="ground_clearance" value="0.0"/>
-    <!-- base_link is aligned with wheel hubs (axle plane).
-         Wheel centers are placed at z=0 in base_link frame. -->
+    <!-- REQUIREMENT:
+         base_link z-axis plane equals wheel hub plane:
+         wheel centers must be at the same z as base_link => wheel_z = 0 -->
     <xacro:property name="wheel_z" value="0.0"/>
     <!-- Joint dynamics -->
@@ -40,5 +34,5 @@
     <!-- ========================= -->
     <link name="${prefix}base_footprint"/>
-    <!-- base_link is at wheel hub height above ground -->
+    <!-- base_link at wheel hub height above ground -->
     <joint name="${prefix}base_footprint_joint" type="fixed">
       <parent link="${prefix}base_footprint"/>
@@ -47,10 +41,10 @@
     </joint>
     <!-- ========================= -->
-    <!-- Base Link (chassis)       -->
+    <!-- Base Link (chassis box)   -->
     <!-- ========================= -->
+    <!-- Box is centered on base_link => box center z == wheel hub z (in base_link frame). -->
     <link name="${prefix}base_link">
       <collision>
-        <!-- Shift chassis geometry upwards so base_link stays on wheel hub plane -->
-        <origin xyz="0 0 ${base_height/2.0}" rpy="0 0 0"/>
+        <origin xyz="0 0 0" rpy="0 0 0"/>
         <geometry>
           <box size="${base_length} ${base_width} ${base_height}"/>
@@ -58,5 +52,5 @@
       </collision>
       <visual>
-        <origin xyz="0 0 ${base_height/2.0}" rpy="0 0 0"/>
+        <origin xyz="0 0 0" rpy="0 0 0"/>
         <geometry>
           <box size="${base_length} ${base_width} ${base_height}"/>
@@ -65,6 +59,5 @@
       </visual>
       <inertial>
-        <!-- Inertial origin aligned with chassis center (same shift as geometry) -->
-        <origin xyz="0 0 ${base_height/2.0}" rpy="0 0 0"/>
+        <origin xyz="0 0 0" rpy="0 0 0"/>
         <mass value="${base_mass}"/>
         <inertia
@@ -118,5 +111,4 @@
     <!-- 4 Wheel Joints            -->
     <!-- ========================= -->
-    <!-- Front-Left -->
     <joint name="${prefix}wheel_fl_joint" type="continuous">
       <parent link="${prefix}base_link"/>
@@ -127,5 +119,4 @@
       <limit effort="${wheel_joint_effort}" velocity="${wheel_joint_velocity}"/>
     </joint>
-    <!-- Front-Right -->
     <joint name="${prefix}wheel_fr_joint" type="continuous">
       <parent link="${prefix}base_link"/>
@@ -136,5 +127,4 @@
       <limit effort="${wheel_joint_effort}" velocity="${wheel_joint_velocity}"/>
     </joint>
-    <!-- Rear-Left -->
     <joint name="${prefix}wheel_rl_joint" type="continuous">
       <parent link="${prefix}base_link"/>
@@ -145,5 +135,4 @@
       <limit effort="${wheel_joint_effort}" velocity="${wheel_joint_velocity}"/>
     </joint>
-    <!-- Rear-Right -->
     <joint name="${prefix}wheel_rr_joint" type="continuous">
       <parent link="${prefix}base_link"/>

Commit message: Add sensor box

File: urdf/mivia_rover_description.urdf.xacro (robot description, xacro)
@@ -2,4 +2,5 @@
 <robot xmlns:xacro="http://www.ros.org/wiki/xacro">
   <xacro:include filename="$(find mivia_rover_description)/urdf/mivia_rover.materials.xacro"/>
+  <xacro:include filename="$(find zed_wrapper)/urdf/zed_descr.urdf.xacro"/>
   <xacro:macro name="mivia_rover" params="prefix">
     <xacro:property name="PI" value="3.1415926535897931"/>
@@ -8,4 +9,13 @@
     <xacro:property name="base_width"  value="0.24"/>
     <xacro:property name="base_height" value="0.10"/>
+    <!-- Sensor box geometry -->
+    <xacro:property name="sensor_box_length" value="0.21"/>
+    <xacro:property name="sensor_box_width"  value="0.17"/>
+    <xacro:property name="sensor_box_height" value="0.075"/>
+    <!--
+      base_sensor_box_offset_z:
+      Vertical space between the base (base_link) and the sensor box along the Z axis.
+    -->
+    <xacro:property name="base_sensor_box_offset_z" value="0.024"/>
     <!-- Base mass/inertia -->
     <xacro:property name="base_mass" value="8.0"/>
@@ -143,4 +153,38 @@
       <limit effort="${wheel_joint_effort}" velocity="${wheel_joint_velocity}"/>
     </joint>
+    <!-- ========================= -->
+    <!-- Sensor Box Link   -->
+    <!-- ========================= -->
+    <link name="${prefix}sensor_box_link">
+      <collision>
+        <origin xyz="0 0 0" rpy="0 0 0"/>
+        <geometry>
+          <box size="${sensor_box_length} ${sensor_box_width} ${sensor_box_height}"/>
+        </geometry>
+      </collision>
+      <visual>
+        <origin xyz="0 0 0" rpy="0 0 0"/>
+        <geometry>
+          <box size="${sensor_box_length} ${sensor_box_width} ${sensor_box_height}"/>
+        </geometry>
+        <material name="mivia_gray"/>
+      </visual>
+    </link>
+    <!-- ========================= -->
+    <!-- Sensor Box joint   -->
+    <!-- ========================= -->
+    <joint name="${prefix}sensor_box_joint" type="fixed">
+      <parent link="${prefix}base_link"/>
+      <child  link="${prefix}sensor_box_link"/>
+      <origin xyz="0 0 ${base_height/2 + sensor_box_height/2 + base_sensor_box_offset_z}" rpy="0 0 0"/>
+    </joint>
+    <!-- ========================= -->
+    <!-- Camera Joint   -->
+    <!-- ========================= -->
+    <joint name="${prefix}camera_joint" type="fixed">
+      <parent link="${prefix}sensor_box_link"/>
+      <child  link="zed_camera_link"/>
+      <origin xyz="0 0 ${sensor_box_height/2}" rpy="0 0 0"/>
+    </joint>
   </xacro:macro>
 </robot>

Commit message: Adding uwb link

File: urdf/mivia_rover_description.urdf.xacro (robot description, xacro)
@@ -18,4 +18,8 @@
     -->
     <xacro:property name="base_sensor_box_offset_z" value="0.024"/>
+    <!-- Uwb geometry -->
+    <xacro:property name="uwb_length" value="0.023"/>
+    <xacro:property name="uwb_width"  value="0.048"/>
+    <xacro:property name="uwb_height" value="0.094"/>
     <!-- Base mass/inertia -->
     <xacro:property name="base_mass" value="8.0"/>
@@ -187,4 +191,30 @@
       <origin xyz="0 0 ${sensor_box_height/2}" rpy="0 0 0"/>
     </joint>
+    <!-- ========================= -->
+    <!-- Uwb Link   -->
+    <!-- ========================= -->
+    <link name="${prefix}uwb_link">
+      <collision>
+        <origin xyz="0 0 0" rpy="0 0 0"/>
+        <geometry>
+          <box size="${uwb_length} ${uwb_width} ${uwb_height}"/>
+        </geometry>
+      </collision>
+      <visual>
+        <origin xyz="0 0 0" rpy="0 0 0"/>
+        <geometry>
+          <box size="${uwb_length} ${uwb_width} ${uwb_height}"/>
+        </geometry>
+        <material name="mivia_gray"/>
+      </visual>
+    </link>
+    <!-- ========================= -->
+    <!-- Uwb joint   -->
+    <!-- ========================= -->
+    <joint name="${prefix}uwb_joint" type="fixed">
+      <parent link="${prefix}sensor_box_link"/>
+      <child  link="${prefix}uwb_link"/>
+      <origin xyz="0.10 0 ${sensor_box_height/2 + uwb_height/2}" rpy="0 0 0"/>
+    </joint>
   </xacro:macro>
 </robot>

Commit message: Editing camera and uwb position

File: urdf/mivia_rover_description.urdf.xacro (robot description, xacro)
@@ -189,5 +189,5 @@
       <parent link="${prefix}sensor_box_link"/>
       <child  link="zed_camera_link"/>
-      <origin xyz="0 0 ${sensor_box_height/2}" rpy="0 0 0"/>
+      <origin xyz="${sensor_box_length/2 - 0.016} 0 ${sensor_box_height/2}" rpy="0 0 0"/>
     </joint>
     <!-- ========================= -->
@@ -215,5 +215,5 @@
       <parent link="${prefix}sensor_box_link"/>
       <child  link="${prefix}uwb_link"/>
-      <origin xyz="0.10 0 ${sensor_box_height/2 + uwb_height/2}" rpy="0 0 0"/>
+      <origin xyz="${sensor_box_length/2 + uwb_length/2} ${sensor_box_width/2 + uwb_width/2 - 0.0661} 0" rpy="0 0 0"/>
     </joint>
   </xacro:macro>
