Commit message: smaller wheel adjusted

File: urdf/mivia_rover_description.urdf.xacro (robot description, xacro)
@@ -25,10 +25,10 @@
     <xacro:property name="base_mass" value="8.0"/>
     <!-- Wheel geometry -->
-    <xacro:property name="wheel_radius" value="0.085"/>
-    <xacro:property name="wheel_width"  value="0.08"/>
+    <xacro:property name="wheel_radius" value="0.07673"/>
+    <xacro:property name="wheel_width"  value="0.08255"/>
     <!-- Wheel mass/inertia -->
     <xacro:property name="wheel_mass" value="0.8"/>
     <!-- Wheel placement -->
-    <xacro:property name="wheelbase" value="0.216"/>
+    <xacro:property name="wheelbase" value="0.219"/>
     <xacro:property name="track"     value="0.355"/>
     <!-- Optional clearance of wheel contact point w.r.t. base_footprint -->

Commit message: separation in config e urdf

File: urdf/mivia_rover_description.urdf.xacro (robot description, xacro)
@@ -3,4 +3,10 @@
   <xacro:include filename="$(find mivia_rover_description)/urdf/mivia_rover.materials.xacro"/>
   <xacro:include filename="$(find zed_wrapper)/urdf/zed_descr.urdf.xacro"/>
+  <!-- Sensor extrinsics (position/orientation of sensor_box, camera, uwb, imu).
+       Kept in a separate yaml so they can be re-measured/tuned without
+       touching URDF syntax. Override config_dir to point at a different
+       calibration directory (e.g. per-unit calibration) if ever needed. -->
+  <xacro:arg name="config_dir" default="$(find mivia_rover_description)"/>
+  <xacro:property name="calibration" value="${xacro.load_yaml('$(arg config_dir)/config/sensors_calibration.yaml')}"/>
   <xacro:macro name="mivia_rover" params="prefix">
     <xacro:property name="PI" value="3.1415926535897931"/>
@@ -13,9 +19,4 @@
     <xacro:property name="sensor_box_width"  value="0.17"/>
     <xacro:property name="sensor_box_height" value="0.075"/>
-    <!--
-      base_sensor_box_offset_z:
-      Vertical space between the base (base_link) and the sensor box along the Z axis.
-    -->
-    <xacro:property name="base_sensor_box_offset_z" value="0.024"/>
     <!-- Uwb geometry -->
     <xacro:property name="uwb_length" value="0.023"/>
@@ -181,39 +182,41 @@
       <parent link="${prefix}base_link"/>
       <child  link="${prefix}sensor_box_link"/>
-      <origin xyz="0 0 ${base_height/2 + sensor_box_height/2 + base_sensor_box_offset_z}" rpy="0 0 0"/>
-    </joint>
-    <!-- ========================= -->
-    <!-- Camera Joint   -->
-    <!-- ========================= -->
+      <origin
+        xyz="${calibration['base_link2sensor_box']['x']} ${calibration['base_link2sensor_box']['y']} ${calibration['base_link2sensor_box']['z']}"
+        rpy="${calibration['base_link2sensor_box']['roll']} ${calibration['base_link2sensor_box']['pitch']} ${calibration['base_link2sensor_box']['yaw']}"/>
+    </joint>
+    <!-- ========================= -->
+    <!-- Camera Link + Joint       -->
+    <!-- ========================= -->
+    <link name="zed_camera_link"/>
     <joint name="${prefix}camera_joint" type="fixed">
       <parent link="${prefix}sensor_box_link"/>
       <child  link="zed_camera_link"/>
-      <origin xyz="${sensor_box_length/2 - 0.016} 0 ${sensor_box_height/2}" rpy="0 0 0"/>
-    </joint>
-    <!-- ========================= -->
-    <!-- Uwb Link   -->
-    <!-- ========================= -->
-    <link name="${prefix}uwb_link">
-      <collision>
-        <origin xyz="0 0 0" rpy="0 0 0"/>
-        <geometry>
-          <box size="${uwb_length} ${uwb_width} ${uwb_height}"/>
-        </geometry>
-      </collision>
-      <visual>
-        <origin xyz="0 0 0" rpy="0 0 0"/>
-        <geometry>
-          <box size="${uwb_length} ${uwb_width} ${uwb_height}"/>
-        </geometry>
-        <material name="mivia_gray"/>
-      </visual>
-    </link>
-    <!-- ========================= -->
-    <!-- Uwb joint   -->
-    <!-- ========================= -->
+      <origin
+        xyz="${calibration['sensor_box2zed_camera']['x']} ${calibration['sensor_box2zed_camera']['y']} ${calibration['sensor_box2zed_camera']['z']}"
+        rpy="${calibration['sensor_box2zed_camera']['roll']} ${calibration['sensor_box2zed_camera']['pitch']} ${calibration['sensor_box2zed_camera']['yaw']}"/>
+    </joint>
+    <!-- ========================= -->
+    <!-- Uwb Link + Joint          -->
+    <!-- ========================= -->
+    <link name="${prefix}uwb_link"/>
     <joint name="${prefix}uwb_joint" type="fixed">
       <parent link="${prefix}sensor_box_link"/>
       <child  link="${prefix}uwb_link"/>
-      <origin xyz="${sensor_box_length/2 + uwb_length/2} ${sensor_box_width/2 + uwb_width/2 - 0.0661} 0" rpy="0 0 0"/>
+      <origin
+        xyz="${calibration['sensor_box2uwb']['x']} ${calibration['sensor_box2uwb']['y']} ${calibration['sensor_box2uwb']['z']}"
+        rpy="${calibration['sensor_box2uwb']['roll']} ${calibration['sensor_box2uwb']['pitch']} ${calibration['sensor_box2uwb']['yaw']}"/>
+    </joint>
+    <!-- ========================= -->
+    <!-- Imu (Xsens MTi-8) Link + Joint -->
+    <!-- ========================= -->
+    <!-- xsens_mti_node.yaml must keep frame_id == "imu_link" (its default) for this to line up. -->
+    <link name="${prefix}imu_link"/>
+    <joint name="${prefix}imu_joint" type="fixed">
+      <parent link="${prefix}sensor_box_link"/>
+      <child  link="${prefix}imu_link"/>
+      <origin
+        xyz="${calibration['sensor_box2imu']['x']} ${calibration['sensor_box2imu']['y']} ${calibration['sensor_box2imu']['z']}"
+        rpy="${calibration['sensor_box2imu']['roll']} ${calibration['sensor_box2imu']['pitch']} ${calibration['sensor_box2imu']['yaw']}"/>
     </joint>
   </xacro:macro>

Commit message: Add Velodyne VLP-16 link and extrinsics
New "velodyne" link fixed to sensor_box_link, with a sensor_box2velodyne
entry in sensors_calibration.yaml (zeros for now, not yet measured).

File: urdf/mivia_rover_description.urdf.xacro (robot description, xacro)
@@ -220,4 +220,17 @@
         rpy="${calibration['sensor_box2imu']['roll']} ${calibration['sensor_box2imu']['pitch']} ${calibration['sensor_box2imu']['yaw']}"/>
     </joint>
+    <!-- ========================= -->
+    <!-- Velodyne VLP-16 Link + Joint -->
+    <!-- ========================= -->
+    <!-- velodyne_vlp16.yaml (mivia_rover_sensing_bringup) must keep
+         frame_id == "velodyne" for the point cloud to line up with this link. -->
+    <link name="${prefix}velodyne"/>
+    <joint name="${prefix}velodyne_joint" type="fixed">
+      <parent link="${prefix}sensor_box_link"/>
+      <child  link="${prefix}velodyne"/>
+      <origin
+        xyz="${calibration['sensor_box2velodyne']['x']} ${calibration['sensor_box2velodyne']['y']} ${calibration['sensor_box2velodyne']['z']}"
+        rpy="${calibration['sensor_box2velodyne']['roll']} ${calibration['sensor_box2velodyne']['pitch']} ${calibration['sensor_box2velodyne']['yaw']}"/>
+    </joint>
   </xacro:macro>
 </robot>
